File: LAB 4/LAB 4.kicad_sch (KiCad schematic)
At the start: 6 parts, among them SW1 SW_SPDT

Commit message: Lab 6
Parts:
- C1: footprint (none) -> Capacitor_THT:C_Radial_D5.0mm_H5.0mm_P2.00mm
- D1: footprint (none) -> LED_THT:LED_D5.0mm
- R1, R2: footprint (none) -> Resistor_THT:R_Axial_DIN0516_L15.5mm_D5.0mm_P20.32mm_Horizontal
- SW1: footprint (none) -> Button_Switch_THT:SW_E-Switch_EG1224_SPDT_Angled
- V1: footprint (none) -> Connector_JST:JST_PH_B2B-PH-K_1x02_P2.00mm_Vertical
Changed lines of the file:
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@@
     (property "Reference" "V1" (id 0) (at 111.125 73.66 0))
     (property "Value" "+9V" (id 1) (at 111.125 76.2 0))
-    (property "Footprint" "" (id 2) (at 110.49 78.74 0)
+    (property "Footprint" "Connector_JST:JST_PH_B2B-PH-K_1x02_P2.00mm_Vertical" (id 2) (at 110.49 78.74 0)
       (effects (font (size 1.27 1.27)) hide)
     )
@@
   )
   (symbol (lib_id "Switch:SW_SPDT") (at 137.16 67.31 0) (unit 1)
-    (in_bom yes) (on_board yes) (fields_autoplaced)
+    (in_bom yes) (on_board yes)
     (property "Reference" "SW1" (id 0) (at 137.16 59.69 0))
     (property "Value" "SW_SPDT" (id 1) (at 137.16 62.23 0))
-    (property "Footprint" "" (id 2) (at 137.16 67.31 0)
-      (effects (font (size 1.27 1.27)) hide)
-    )
+    (property "Footprint" "Button_Switch_THT:SW_E-Switch_EG1224_SPDT_Angled" (id 2) (at 140.97 48.26 0))
     (property "Datasheet" "~" (id 3) (at 137.16 67.31 0)
       (effects (font (size 1.27 1.27)) hide)
@@
   )
   (symbol (lib_id "Device:R") (at 120.65 67.31 90) (unit 1)
-    (in_bom yes) (on_board yes) (fields_autoplaced)
+    (in_bom yes) (on_board yes)
     (property "Reference" "R2" (id 0) (at 120.65 60.96 90))
     (property "Value" "2.2k" (id 1) (at 120.65 63.5 90))
-    (property "Footprint" "" (id 2) (at 120.65 69.088 90)
-      (effects (font (size 1.27 1.27)) hide)
-    )
+    (property "Footprint" "Resistor_THT:R_Axial_DIN0516_L15.5mm_D5.0mm_P20.32mm_Horizontal" (id 2) (at 148.59 45.72 90))
     (property "Datasheet" "~" (id 3) (at 120.65 67.31 0)
       (effects (font (size 1.27 1.27)) hide)
@@
   )
   (symbol (lib_id "Device:LED") (at 165.1 83.82 90) (unit 1)
-    (in_bom yes) (on_board yes) (fields_autoplaced)
+    (in_bom yes) (on_board yes)
     (property "Reference" "D1" (id 0) (at 168.91 84.1374 90)
       (effects (font (size 1.27 1.27)) (justify right))
@@
       (effects (font (size 1.27 1.27)) (justify right))
     )
-    (property "Footprint" "" (id 2) (at 165.1 83.82 0)
-      (effects (font (size 1.27 1.27)) hide)
-    )
+    (property "Footprint" "LED_THT:LED_D5.0mm" (id 2) (at 180.34 86.36 0))
     (property "Datasheet" "~" (id 3) (at 165.1 83.82 0)
       (effects (font (size 1.27 1.27)) hide)
@@
   )
   (symbol (lib_id "Device:C") (at 143.51 78.74 0) (unit 1)
-    (in_bom yes) (on_board yes) (fields_autoplaced)
+    (in_bom yes) (on_board yes)
     (property "Reference" "C1" (id 0) (at 147.32 77.4699 0)
       (effects (font (size 1.27 1.27)) (justify left))
@@
       (effects (font (size 1.27 1.27)) (justify left))
     )
-    (property "Footprint" "" (id 2) (at 144.4752 82.55 0)
-      (effects (font (size 1.27 1.27)) hide)
-    )
+    (property "Footprint" "Capacitor_THT:C_Radial_D5.0mm_H5.0mm_P2.00mm" (id 2) (at 140.97 50.8 0))
     (property "Datasheet" "~" (id 3) (at 143.51 78.74 0)
       (effects (font (size 1.27 1.27)) hide)
@@
   )
   (symbol (lib_id "Device:R") (at 165.1 73.66 180) (unit 1)
-    (in_bom yes) (on_board yes) (fields_autoplaced)
+    (in_bom yes) (on_board yes)
     (property "Reference" "R1" (id 0) (at 167.64 72.3899 0)
       (effects (font (size 1.27 1.27)) (justify right))
@@
       (effects (font (size 1.27 1.27)) (justify right))
     )
-    (property "Footprint" "" (id 2) (at 166.878 73.66 90)
-      (effects (font (size 1.27 1.27)) hide)
-    )
+    (property "Footprint" "Resistor_THT:R_Axial_DIN0516_L15.5mm_D5.0mm_P20.32mm_Horizontal" (id 2) (at 185.42 74.93 90))
     (property "Datasheet" "~" (id 3) (at 165.1 73.66 0)
       (effects (font (size 1.27 1.27)) hide)
@@
   (symbol_instances
     (path "/e9be0c2e-757e-4f0d-b4ca-03db2efd0331"
-      (reference "C1") (unit 1) (value "C") (footprint "")
+      (reference "C1") (unit 1) (value "C") (footprint "Capacitor_THT:C_Radial_D5.0mm_H5.0mm_P2.00mm")
     )
     (path "/d0aa26bd-25c6-4084-8fea-c8f6ead61260"
-      (reference "D1") (unit 1) (value "LED") (footprint "")
+      (reference "D1") (unit 1) (value "LED") (footprint "LED_THT:LED_D5.0mm")
     )
     (path "/fffe3066-8f36-4c2a-abca-660ad13066e8"
-      (reference "R1") (unit 1) (value "20k") (footprint "")
+      (reference "R1") (unit 1) (value "20k") (footprint "Resistor_THT:R_Axial_DIN0516_L15.5mm_D5.0mm_P20.32mm_Horizontal")
     )
     (path "/cc34ccc1-7023-45a9-a238-c59ba9fed633"
-      (reference "R2") (unit 1) (value "2.2k") (footprint "")
+      (reference "R2") (unit 1) (value "2.2k") (footprint "Resistor_THT:R_Axial_DIN0516_L15.5mm_D5.0mm_P20.32mm_Horizontal")
     )
     (path "/18d02db9-0337-45c5-bb89-1f213e9128f2"
-      (reference "SW1") (unit 1) (value "SW_SPDT") (footprint "")
+      (reference "SW1") (unit 1) (value "SW_SPDT") (footprint "Button_Switch_THT:SW_E-Switch_EG1224_SPDT_Angled")
     )
     (path "/0aa285b0-ab96-4259-a38d-99c6fe498b8a"
-      (reference "V1") (unit 1) (value "+9V") (footprint "")
+      (reference "V1") (unit 1) (value "+9V") (footprint "Connector_JST:JST_PH_B2B-PH-K_1x02_P2.00mm_Vertical")
     )
   )
