File: lab4/LAB 4.kicad_sch (KiCad schematic)
At the start: 6 parts, among them SW1 SW_SPDT

Commit message: Add files via upload
Parts:
- C1: value C -> 4.7 microF
Changed lines of the file:
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@@
       (effects (font (size 1.27 1.27)) (justify left))
     )
-    (property "Value" "C" (id 1) (at 147.32 80.0099 0)
+    (property "Value" "4.7 microF" (id 1) (at 147.32 80.0099 0)
       (effects (font (size 1.27 1.27)) (justify left))
     )
@@
   (symbol_instances
     (path "/e9be0c2e-757e-4f0d-b4ca-03db2efd0331"
-      (reference "C1") (unit 1) (value "C") (footprint "")
+      (reference "C1") (unit 1) (value "4.7 microF") (footprint "")
     )
     (path "/d0aa26bd-25c6-4084-8fea-c8f6ead61260"
